Commit message: Added working laser and pan

File: pr2_description/urdf/head_v0/head.transmission.xacro (robot description, xacro)
@@ -8,8 +8,8 @@
     <type>transmission_interface/SimpleTransmission</type>
     <joint name="${name}_joint">
-      <hardwareInterface>hardware_interface/PositionJointInterface</hardwareInterface>
+      <hardwareInterface>hardware_interface/EffortJointInterface</hardwareInterface>
     </joint>
     <actuator name="${name}_motor">
-      <hardwareInterface>hardware_interface/PositionJointInterface</hardwareInterface>
+      <hardwareInterface>hardware_interface/EffortJointInterface</hardwareInterface>
       <mechanicalReduction>1.0</mechanicalReduction>
     </actuator>
@@ -20,8 +20,8 @@
     <type>transmission_interface/SimpleTransmission</type>
     <joint name="${name}_joint">
-      <hardwareInterface>hardware_interface/PositionJointInterface</hardwareInterface>
+      <hardwareInterface>hardware_interface/EffortJointInterface</hardwareInterface>
     </joint>
     <actuator name="${name}_motor">
-      <hardwareInterface>hardware_interface/PositionJointInterface</hardwareInterface>
+      <hardwareInterface>hardware_interface/EffortJointInterface</hardwareInterface>
       <mechanicalReduction>1.0</mechanicalReduction>
     </actuator>

File: pr2_description/urdf/head_v0/head.urdf.xacro (robot description, xacro)
@@ -28,5 +28,5 @@
         <origin xyz="0 0 0.0" rpy="0 0 0 " />
         <geometry>
-          <mesh filename="package://pr2_description/meshes/head_v0/head_pan.dae"  />
+          <mesh filename="package://pr2_description/meshes/head_v0/head_pan_png.dae"  />
         </geometry>
         <material name="Blue" />
@@ -63,5 +63,5 @@
         <origin xyz="0 0 0" rpy="0.0 0.0 0.0" />
         <geometry>
-          <mesh filename="package://pr2_description/meshes/head_v0/head_tilt.dae"  />
+          <mesh filename="package://pr2_description/meshes/head_v0/head_tilt_green.dae"  />
         </geometry>
         <material name="Green" />

File: pr2_description/urdf/tilting_laser_v0/tilting_laser.transmission.xacro (robot description, xacro)
@@ -8,8 +8,8 @@
     <type>transmission_interface/SimpleTransmission</type>
     <joint name="${name}_mount_joint">
-      <hardwareInterface>hardware_interface/PositionJointInterface</hardwareInterface>
+      <hardwareInterface>hardware_interface/EffortJointInterface</hardwareInterface>
     </joint>
     <actuator name="${name}_mount_motor">
-      <hardwareInterface>hardware_interface/PositionJointInterface</hardwareInterface>
+      <hardwareInterface>hardware_interface/EffortJointInterface</hardwareInterface>
       <mechanicalReduction>1.0</mechanicalReduction>
     </actuator>

File: pr2_description/urdf/tilting_laser_v0/tilting_laser.urdf.xacro (robot description, xacro)
@@ -29,5 +29,5 @@
         <origin xyz="0 0 0" rpy="0 0 0" />
         <geometry>
-          <mesh filename="package://pr2_description/meshes/tilting_laser_v0/tilting_hokuyo.dae" />
+          <mesh filename="package://pr2_description/meshes/tilting_laser_v0/tilting_hokuyo_png.dae" />
         </geometry>
         <material name="Red" />
